File: raspi3-4xWS2812-lvds.sch (KiCad schematic (older format))
At the start: 39 parts, among them J1 Conn_ARM_JTAG_SWD_10, J2 Raspberry_Pi_2_3, J3 Conn_02x08_Odd_Even, J4 Conn_02x04_Odd_Even, J5 Conn_01x02, U1 SAMC21G17A-A, U2 SN65LVDS047D, U3 TJA1049T-3, Y1 8MHz

Commit message: add quad OR gate as level shifter
Parts:
- added C?: 1uF, symbol Device:C_Small
- added U? (x5): 74LS32, symbol 74xx:74LS32
Connections:
- wire segments 151 -> 163

Commit message: annotate U4
Parts:
- gave numbers to parts that had none: 2
Changed lines of the file:
@@
 UART5_TX
 $Comp
-L power:+5V #PWR?
+L power:+5V #PWR0101
 U 1 1 5B61ACCE
 P 5050 5050
-F 0 "#PWR?" H 5050 4900 50  0001 C CNN
+F 0 "#PWR0101" H 5050 4900 50  0001 C CNN
 F 1 "+5V" H 5065 5223 50  0000 C CNN
 F 2 "" H 5050 5050 50  0001 C CNN
@@
 $EndComp
 $Comp
-L power:GND #PWR?
+L power:GND #PWR0102
 U 1 1 5B61AF1F
 P 5050 6050
-F 0 "#PWR?" H 5050 5800 50  0001 C CNN
+F 0 "#PWR0102" H 5050 5800 50  0001 C CNN
 F 1 "GND" H 5055 5877 50  0000 C CNN
 F 2 "" H 5050 6050 50  0001 C CNN
@@
 $EndComp
 $Comp
-L Device:C_Small C?
+L Device:C_Small C15
 U 1 1 5B61B0A4
 P 4550 5550
-F 0 "C?" H 4642 5596 50  0000 L CNN
+F 0 "C15" H 4642 5596 50  0000 L CNN
 F 1 "1uF" H 4642 5505 50  0000 L CNN
 F 2 "" H 4550 5550 50  0001 C CNN
@@
 $EndComp
 $Comp
-L power:GND #PWR?
+L power:GND #PWR0103
 U 1 1 5B61B0AA
 P 4550 5650
-F 0 "#PWR?" H 4550 5400 50  0001 C CNN
+F 0 "#PWR0103" H 4550 5400 50  0001 C CNN
 F 1 "GND" H 4555 5477 50  0000 C CNN
 F 2 "" H 4550 5650 50  0001 C CNN
@@
 $EndComp
 $Comp
-L power:+5V #PWR?
+L power:+5V #PWR0104
 U 1 1 5B61B0B0
 P 4550 5450
-F 0 "#PWR?" H 4550 5300 50  0001 C CNN
+F 0 "#PWR0104" H 4550 5300 50  0001 C CNN
 F 1 "+5V" H 4565 5623 50  0000 C CNN
 F 2 "" H 4550 5450 50  0001 C CNN
@@
 $EndComp
 $Comp
-L 74xx:74LS32 U?
+L 74xx:74LS32 U4
 U 1 1 5B62C263
 P 6000 4900
-F 0 "U?" H 6000 4900 50  0000 C CNN
+F 0 "U4" H 6000 4900 50  0000 C CNN
 F 1 "74LS32" H 6000 4700 50  0000 C CNN
 F 2 "" H 6000 4900 50  0001 C CNN
@@
 $EndComp
 $Comp
-L 74xx:74LS32 U?
+L 74xx:74LS32 U4
 U 2 1 5B62C3FB
 P 6000 5400
-F 0 "U?" H 6000 5400 50  0000 C CNN
+F 0 "U4" H 6000 5400 50  0000 C CNN
 F 1 "74LS32" H 6000 5200 50  0000 C CNN
 F 2 "" H 6000 5400 50  0001 C CNN
@@
 $EndComp
 $Comp
-L 74xx:74LS32 U?
+L 74xx:74LS32 U4
 U 3 1 5B62C4D2
 P 6000 5900
-F 0 "U?" H 6000 5900 50  0000 C CNN
+F 0 "U4" H 6000 5900 50  0000 C CNN
 F 1 "74LS32" H 6000 5700 50  0000 C CNN
 F 2 "" H 6000 5900 50  0001 C CNN
@@
 $EndComp
 $Comp
-L 74xx:74LS32 U?
+L 74xx:74LS32 U4
 U 4 1 5B62C5BE
 P 6000 6400
-F 0 "U?" H 6000 6400 50  0000 C CNN
+F 0 "U4" H 6000 6400 50  0000 C CNN
 F 1 "74LS32" H 6000 6200 50  0000 C CNN
 F 2 "" H 6000 6400 50  0001 C CNN
@@
 $EndComp
 $Comp
-L 74xx:74LS32 U?
+L 74xx:74LS32 U4
 U 5 1 5B62C6BB
 P 5050 5550
-F 0 "U?" H 4800 5900 50  0000 L CNN
+F 0 "U4" H 4800 5900 50  0000 L CNN
 F 1 "74LS32" H 4900 5550 50  0000 L CNN
 F 2 "" H 5050 5550 50  0001 C CNN
@@
 $EndComp
 $Comp
-L power:GND #PWR?
+L power:GND #PWR0105
 U 1 1 5B6325B2
 P 5700 6500
-F 0 "#PWR?" H 5700 6250 50  0001 C CNN
+F 0 "#PWR0105" H 5700 6250 50  0001 C CNN
 F 1 "GND" H 5705 6327 50  0000 C CNN
 F 2 "" H 5700 6500 50  0001 C CNN
@@
 $EndComp
 $Comp
-L power:GND #PWR?
+L power:GND #PWR0106
 U 1 1 5B6327AC
 P 5700 6000
-F 0 "#PWR?" H 5700 5750 50  0001 C CNN
+F 0 "#PWR0106" H 5700 5750 50  0001 C CNN
 F 1 "GND" H 5705 5827 50  0000 C CNN
 F 2 "" H 5700 6000 50  0001 C CNN
@@
 $EndComp
 $Comp
-L power:GND #PWR?
+L power:GND #PWR0107
 U 1 1 5B63286B
 P 5700 5500
-F 0 "#PWR?" H 5700 5250 50  0001 C CNN
+F 0 "#PWR0107" H 5700 5250 50  0001 C CNN
 F 1 "GND" H 5705 5327 50  0000 C CNN
 F 2 "" H 5700 5500 50  0001 C CNN
@@
 $EndComp
 $Comp
-L power:GND #PWR?
+L power:GND #PWR0108
 U 1 1 5B6328D0
 P 5700 5000
-F 0 "#PWR?" H 5700 4750 50  0001 C CNN
+F 0 "#PWR0108" H 5700 4750 50  0001 C CNN
 F 1 "GND" H 5705 4827 50  0000 C CNN
 F 2 "" H 5700 5000 50  0001 C CNN

Commit message: board layout!
Parts:
- C1, C10, C11, C12, C13, C14, C15, C2, C3, C4, C5, C6, C7, C8, C9: footprint (none) -> Capacitor_SMD:C_0603_1608Metric
- D1, D2: footprint (none) -> LED_SMD:LED_0603_1608Metric
- J2: footprint (none) -> Connector_PinHeader_2.54mm:PinHeader_2x20_P2.54mm_Vertical
- J3: footprint (none) -> Connector_PinHeader_2.54mm:PinHeader_2x08_P2.54mm_Horizontal
- J4: footprint (none) -> Connector_PinHeader_2.54mm:PinHeader_2x04_P2.54mm_Vertical
- J5: footprint (none) -> Connector_PinHeader_2.54mm:PinHeader_1x02_P2.54mm_Vertical
- R1, R10, R11, R12, R13, R2, R3, R4, R5, R6, R7, R8, R9: footprint (none) -> Resistor_SMD:R_0603_1608Metric
- R14: footprint (none) -> Resistor_SMD:R_0805_2012Metric
- U4: footprint (none) -> Package_SO:SOIC-14_3.9x8.7mm_P1.27mm
- Y1: footprint (none) -> Crystal:Crystal_SMD_Abracon_ABM3-2Pin_5.0x3.2mm
Connections:
- net labels added: LED0, LED1
- wire segments 163 -> 159
- no-connect marks 38 -> 39
Other:
- moved on the sheet: U1

Commit message: improve silkscreen, make jtag connector through hole
Parts:
- J1: footprint Connector_PinHeader_1.27mm:PinHeader_2x05_P1.27mm_Vertical_SMD -> Connector_PinHeader_1.27mm:PinHeader_2x05_P1.27mm_Vertical
Changed lines of the file:
@@
 F 0 "J1" H 2150 6700 50  0000 R CNN
 F 1 "Conn_ARM_JTAG_SWD_10" V 2000 6600 50  0000 R CNN
-F 2 "Connector_PinHeader_1.27mm:PinHeader_2x05_P1.27mm_Vertical_SMD" H 2500 5600 50  0001 L TNN
+F 2 "Connector_PinHeader_1.27mm:PinHeader_2x05_P1.27mm_Vertical" H 2500 5600 50  0001 L TNN
 F 3 "http://infocenter.arm.com/help/topic/com.arm.doc.faqs/attached/13634/cortex_debug_connectors.pdf" V 2100 4900 50  0001 C CNN
 	1    2450 6150
